Commit message: update obstacles and pcd save files

File: envs/models/obstacles/high_table.urdf (robot description, URDF)
Before this commit: robot plane, 5 links, 4 joints
Links:
- link link_leg1: geometry collision mesh filename=mesh/high_table/link_leg1.obj; visual mesh filename=mesh/high_table/link_leg1.obj
- link link_leg2: geometry collision mesh filename=mesh/high_table/link_leg2.obj; visual mesh filename=mesh/high_table/link_leg2.obj
- link link_leg3: geometry collision mesh filename=mesh/high_table/link_leg3.obj; visual mesh filename=mesh/high_table/link_leg3.obj
- link link_leg4: geometry collision mesh filename=mesh/high_table/link_leg4.obj; visual mesh filename=mesh/high_table/link_leg4.obj
- link link_plane: geometry collision mesh filename=mesh/high_table/link_plane.obj; visual mesh filename=mesh/high_table/link_plane.obj

File: envs/models/obstacles/low_table.urdf (robot description, URDF)
Before this commit: robot plane, 5 links, 4 joints
Links:
- link link_leg1: geometry collision mesh filename=mesh/low_table/link_leg1.obj; visual mesh filename=mesh/low_table/link_leg1.obj
- link link_leg2: geometry collision mesh filename=mesh/low_table/link_leg2.obj; visual mesh filename=mesh/low_table/link_leg2.obj
- link link_leg3: geometry collision mesh filename=mesh/low_table/link_leg3.obj; visual mesh filename=mesh/low_table/link_leg3.obj
- link link_leg4: geometry collision mesh filename=mesh/low_table/link_leg4.obj; visual mesh filename=mesh/low_table/link_leg4.obj
- link link_plane: geometry collision mesh filename=mesh/low_table/link_plane.obj; visual mesh filename=mesh/low_table/link_plane.obj

File: envs/models/obstacles/shelve.urdf (robot description, URDF)
Before this commit: robot plane, 6 links, 5 joints
Links:
- link shelve_back: geometry collision mesh filename=mesh/shelve/shelve_back.obj; visual mesh filename=mesh/shelve/shelve_back.obj
- link shelve_bottom: geometry collision mesh filename=mesh/shelve/shelve_bottom.obj; visual mesh filename=mesh/shelve/shelve_bottom.obj
- link shelve_left: geometry collision mesh filename=mesh/shelve/shelve_left.obj; visual mesh filename=mesh/shelve/shelve_left.obj
- link shelve_middle: geometry collision mesh filename=mesh/shelve/shelve_middle.obj; visual mesh filename=mesh/shelve/shelve_middle.obj
- link shelve_right: geometry collision mesh filename=mesh/shelve/shelve_right.obj; visual mesh filename=mesh/shelve/shelve_right.obj
- link shelve_upper: geometry collision mesh filename=mesh/shelve/shelve_upper.obj; visual mesh filename=mesh/shelve/shelve_upper.obj

Commit message: set convension for mesh file name

File: envs/models/obstacles/high_table.urdf (robot description, URDF)
Before this commit: robot plane, 5 links, 4 joints
Links:
- removed link link_leg1
- removed link link_leg2
- removed link link_leg3
- removed link link_leg4
- removed link link_plane
- added link high_table_leg1, mass .0; collision mesh filename=mesh/high_table/high_table_leg1.obj; visual mesh filename=mesh/high_table/high_table_leg1.obj
- added link high_table_leg2, mass .0; collision mesh filename=mesh/high_table/high_table_leg2.obj; visual mesh filename=mesh/high_table/high_table_leg2.obj
- added link high_table_leg3, mass .0; collision mesh filename=mesh/high_table/high_table_leg3.obj; visual mesh filename=mesh/high_table/high_table_leg3.obj
- added link high_table_leg4, mass .0; collision mesh filename=mesh/high_table/high_table_leg4.obj; visual mesh filename=mesh/high_table/high_table_leg4.obj
- added link high_table_plane, mass .0; collision mesh filename=mesh/high_table/high_table_plane.obj; visual mesh filename=mesh/high_table/high_table_plane.obj
Joints:
- joint fixed_joint1: child link_leg1 -> high_table_leg1; parent link_plane -> high_table_plane
- joint fixed_joint2: child link_leg2 -> high_table_leg2; parent link_plane -> high_table_plane
- joint fixed_joint3: child link_leg3 -> high_table_leg3; parent link_plane -> high_table_plane
- joint fixed_joint4: child link_leg4 -> high_table_leg4; parent link_plane -> high_table_plane

File: envs/models/obstacles/low_table.urdf (robot description, URDF)
Before this commit: robot plane, 5 links, 4 joints
Links:
- removed link link_leg1
- removed link link_leg2
- removed link link_leg3
- removed link link_leg4
- removed link link_plane
- added link low_table_leg1, mass .0; collision mesh filename=mesh/low_table/low_table_leg1.obj; visual mesh filename=mesh/low_table/low_table_leg1.obj
- added link low_table_leg2, mass .0; collision mesh filename=mesh/low_table/low_table_leg2.obj; visual mesh filename=mesh/low_table/low_table_leg2.obj
- added link low_table_leg3, mass .0; collision mesh filename=mesh/low_table/low_table_leg3.obj; visual mesh filename=mesh/low_table/low_table_leg3.obj
- added link low_table_leg4, mass .0; collision mesh filename=mesh/low_table/low_table_leg4.obj; visual mesh filename=mesh/low_table/low_table_leg4.obj
- added link low_table_plane, mass .0; collision mesh filename=mesh/low_table/low_table_plane.obj; visual mesh filename=mesh/low_table/low_table_plane.obj
Joints:
- joint fixed_joint1: child link_leg1 -> low_table_leg1; parent link_plane -> low_table_plane
- joint fixed_joint2: child link_leg2 -> low_table_leg2; parent link_plane -> low_table_plane
- joint fixed_joint3: child link_leg3 -> low_table_leg3; parent link_plane -> low_table_plane
- joint fixed_joint4: child link_leg4 -> low_table_leg4; parent link_plane -> low_table_plane
