Commit message: TrapBoxScaled

File: envs/models/obstacles/trapezoid_box.urdf (robot description, URDF)
Before this commit: robot Box, 5 links, 4 joints
Links:
- removed link base_link
- removed link wing_1
- removed link wing_2
- removed link wing_3
- removed link wing_4
- added link trapbox_base_link, mass 0; collision mesh filename=mesh/trapezoid_box/trapbox_base_link.obj; visual mesh filename=mesh/trapezoid_box/trapbox_base_link.obj
- added link trapbox_wing_1, mass 0; collision mesh filename=mesh/trapezoid_box/trapbox_wing_1.obj; visual mesh filename=mesh/trapezoid_box/trapbox_wing_1.obj
- added link trapbox_wing_2, mass 0; collision mesh filename=mesh/trapezoid_box/trapbox_wing_2.obj; visual mesh filename=mesh/trapezoid_box/trapbox_wing_2.obj
- added link trapbox_wing_3, mass 0; collision mesh filename=mesh/trapezoid_box/trapbox_wing_3.obj; visual mesh filename=mesh/trapezoid_box/trapbox_wing_3.obj
- added link trapbox_wing_4, mass 0; collision mesh filename=mesh/trapezoid_box/trapbox_wing_4.obj; visual mesh filename=mesh/trapezoid_box/trapbox_wing_4.obj
Joints:
- joint fixed_joint1: child wing_1 -> trapbox_wing_1; parent base_link -> trapbox_base_link
- joint fixed_joint2: child wing_2 -> trapbox_wing_2; parent base_link -> trapbox_base_link
- joint fixed_joint3: child wing_3 -> trapbox_wing_3; parent base_link -> trapbox_base_link
- joint fixed_joint4: child wing_4 -> trapbox_wing_4; parent base_link -> trapbox_base_link
