Commit message: onearm with box env added

File: envs/models/obstacles/box4.urdf (robot description, URDF)
Before this commit: robot boxobs, 1 links, 0 joints
Links:
- removed link boxobsLink
- added link box1link, mass .0; collision mesh filename=mesh/box/box4.obj; visual mesh filename=mesh/box/box4.obj
